File: hardware/02-midi-cv/kicad/sam17-midicv.kicad_sch (KiCad schematic)
At the start: 42 parts, among them J1 BUS +12/G/G/-12, J2 +5V/RTN (mod.1 J6), J3 RPi 3B+ GPIO, J4 CV1, J5 CV2, J6 CV3, J7 GATE_OUT, J8 LCD 16x2 HD44780, Q1 2N7002, Q2 2N7002, SW1 UP, SW2 DOWN, SW3 BACK, SW4 ENTER, U1 AD5686RBRUZ, U2 TL074H

Commit message: Modulo 2: colocacion y masas partidas de la PCB (17 redes sin rutear)
TANDA INCOMPLETA A PROPOSITO, y marcada como tal: build_pcb.py sale con
codigo 2 mientras queden redes sin rutear, para que nadie confunda esto
con una placa fabricable.

LO QUE SI ESTA CERRADO Y VERIFICADO

  colocacion .............. 44 huellas, nada fuera de placa, sin solapes
  frontera de masas ....... 4.00 mm de hueco MEDIDO sobre el cobre relleno
  plano analogico ......... una sola isla, ninguna pista lo parte
  cada pieza en su lado ... verificado pad a pad
  DRC ..................... 0 infracciones sobre lo ruteado
  ruteado ................. 134 segmentos, 26 vias

LO QUE FALTA: 17 redes, casi todas del lado digital (las seis del LCD,
los botones, el SPI cruzando a la frontera). No son culpa del ruteador
sino de la congestion de ese lado.

LA REGLA DE LA PLACA

Frontera vertical en x=78: GNDD a la izquierda, GNDA a la derecha, 4 mm
sin cobre en B.Cu entre medias. Lo que cruza son senales por F.Cu, que
pasan POR ENCIMA del hueco sin unir las masas.

El DAC vive justo en la frontera a proposito y va GIRADO 180 para que sus
patillas de SPI miren al Pi y las analogicas al amplificador; sin girarlo
el SPI tiene que rodear el chip entero.

Asimetria deliberada: el plano DIGITAL puede fragmentarse, el ANALOGICO
no. Alli el plano no mide nada, aqui sostiene el presupuesto de
afinacion. La comprobacion cuenta las islas del vertido analogico y exige
exactamente una. La primera version prohibia toda pista por B.Cu en ese
lado, que era un proxy y de los malos: lo que hace dano no es que haya
cobre abajo, es que el plano quede PARTIDO.

UN ERROR DEL ESQUEMATICO QUE DESTAPO LA COLOCACION

C4 desacoplaba el +3V3 (riel digital) contra la masa ANALOGICA. Mirandolo,
el reparto entero estaba mal y ademas al DAC le faltaba desacoplo local.
Ahora: C1/C2 (+-12 V) contra GNDA, C3/C4 (+5 V y +3V3) contra GNDD junto a
su conector, y C5/C6/C7 pegados al DAC contra GNDA, que es la masa del
propio chip — la corrie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
Parts:
- added C6, C7: 100n, Capacitor_THT:C_Disc_D5.0mm_W2.5mm_P5.00mm, symbol Device:C
Connections:
- net +3V3: now also C7.1
- net +5V: now also C6.1
- net GNDA: now also C6.2, C7.2; no longer C3.2, C4.2
- net GNDD: now also C3.2, C4.2
