File: hardware/01-power-supply/v2/kicad/sam17-power-v2.kicad_pcb (KiCad board)
At the start: 2 copper layers, 150 x 200 mm, 85 parts, among them J1 TerminalBlock_MaiXu_MX126-5.0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, J2 Molex_KK-254_AE-6410-04A_1x04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, J3 TerminalBlock_MaiXu_MX126-5.0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, J4 TerminalBlock_MaiXu_MX126-5.0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, J5 Faston_6.3x0.8mm_PCB_2Leg_P5.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, J6 Molex_KK-254_AE-6410-02A_1x02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, J7 TerminalBlock_MaiXu_MX126-5.0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, Q1 TO-92_Inline_Wide, U1 TO-220-5_Vertical, U2 TO-220-5_Vertical, U3 TO-220-3_Vertical, U4 DFN-10-1EP_3x3mm_P0.5mm_EP1.6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, U5 DFN-10-1EP_3x3mm_P0.5mm_EP1.6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, U6 DFN-12-1EP_3x3mm_P0.45mm_EP1.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, U7 DFN-12-1EP_3x3mm_P0.45mm_EP1.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

Commit message: fix(hw/psu-v2): ola review fase C -- silk BR1/TP/J2/U2, pads U1/U2 anchos, Val real en pos.csv
F1: marca "+" real junto al pad 1 de BR1 en F.SilkS (la huella stock es
simetrica, no traia cruz). F2: 16 textos libres de serigrafia que la placa
no tenia -- titulo+rev, señal de cada TP (leida del netlist real), aviso
"U2 TAB = VRAW- MICA" junto a su disipador, y polaridades de J2 (orden real
del netlist: -12V/GND/GND/+12V, no el orden intuitivo). F3: pads THT de
U1/U2 ensanchados a 1.4x1.8mm -- resuelve (no bendice) las 10 violaciones
annular_width que traia el DRC. F4/F5: documentacion en fab/README.md
(vias de EP abiertas en pasta) y design-notes.md §3.2 (asimetria termica
intra-pareja de las granjas EP), sin tocar routing. F6: corrige comentario
obsoleto sobre el footprint _ThermalVias que U6/U7 nunca usaron. F7:
pos.csv ya trae el Value real del BOM en vez del nombre de la huella.

Pipeline completo re-verificado: ERC 0 errores, check_bom.py OK, DRC real
en 0 infracciones y 0 sin conectar (antes: 10 annular_width "aceptadas").
Fab (gerbers/drill/pos/bom-jlc) y renders 3D regenerados desde el PCB
nuevo.

Co-Authored-By: Claude Fable 5 <noreply@anthropic.com>
Claude-Session: https://claude.ai/code/session_01Xqa4XDcufx4ptQE2gEAZoo
Parts:
- BR1: value Diode_Bridge_DIP-4_W7.62mm_P5.08mm -> DB207
- C1, C12, C13, C2: value CP_Radial_D16.0mm_P7.50mm -> 4700uF/25V electrolitico
- C10: value CP_Radial_D6.3mm_P2.50mm -> 100uF/25V electrolitico
- C11: value C_Disc_D5.0mm_W2.5mm_P5.00mm -> 0.1uF ceramico
- C14: value C_Disc_D5.0mm_W2.5mm_P5.00mm -> 100nF ceramico
- C15, C16: value C_1210_3225Metric -> 22 uF X7R baja fuga 25 V 1210
- C17, C18: value CP_Radial_D6.3mm_P2.50mm -> 22 uF
- C19, C20, C21, C22, C23, C24, C25, C26: value C_1206_3216Metric -> 10 uF X7R 50 V
- C27, C28: value C_Disc_D5.0mm_W2.5mm_P5.00mm -> 0.47 uF ceramico
- C9: value C_Disc_D5.0mm_W2.5mm_P5.00mm -> 0.33uF ceramico
- D10, D11: value D_SMA -> SS14
- D12, D13, D5: value D_DO-41_SOD81_P10.16mm_Horizontal -> 1N4001
- D3: value LED_D3.0mm -> LED rojo 3mm
- D4: value LED_D3.0mm -> LED amarillo 3mm
- D6: value LED_D3.0mm -> LED verde 3mm
- D7: value D_DO-35_SOD27_P7.62mm_Horizontal -> BZX55C15
- D8, D9: value D_SMA -> SMAJ15A
- F1: value Fuseholder_Cylinder-5x20mm_Schurter_FPG4_Vertical_Closed -> Fusible 1.6A lento + portafusible CERRADO 5x20
- J1, J3: value TerminalBlock_MaiXu_MX126-5.0-03P_1x03_P5.00mm -> Barrier block 3 pos
- J2: value Molex_KK-254_AE-6410-04A_1x04_P2.54mm_Vertical -> Molex KK-254 4 pos
- J4, J7: value TerminalBlock_MaiXu_MX126-5.0-02P_1x02_P5.00mm -> Barrier block 2 pos
- J5: value Faston_6.3x0.8mm_PCB_2Leg_P5.0mm -> Faston macho 6.3mm PCB
- J6: value Molex_KK-254_AE-6410-02A_1x02_P2.54mm_Vertical -> Molex KK-254 2 pos
- JP1: value NetTie-2_SMD_Pad0.5mm -> Net tie GNDREF<->GND
- NT1: value NTC_Disc_D11.5mm_W4.5mm_P7.5mm -> SL10-5R020
- Q1: value TO-92_Inline_Wide -> BT169D
- R1, R2: value R_Axial_DIN0207_L6.3mm_D2.5mm_P10.16mm_Horizontal -> 2.2k 1/4W
- R10, R9: value R_0805_2012Metric -> 120k 0.1% 25ppm thin-film
- R11, R12: value R_0603_1608Metric -> 374 ohm 1%
- R13, R14: value R_0603_1608Metric -> 9.31k 1%
- R15, R16, R17, R18: value R_1206_3216Metric -> 20 mOhm 1%
- R3: value R_Axial_DIN0207_L6.3mm_D2.5mm_P10.16mm_Horizontal -> 680R 1/4W
- R4: value R_Axial_DIN0207_L6.3mm_D2.5mm_P10.16mm_Horizontal -> 1k 1/4W
- R5: value R_Axial_DIN0207_L6.3mm_D2.5mm_P10.16mm_Horizontal -> 8.66k 1% 1/4W
- R6, R8: value R_Axial_DIN0207_L6.3mm_D2.5mm_P10.16mm_Horizontal -> 1k 1% 1/4W
- R7: value R_Axial_DIN0207_L6.3mm_D2.5mm_P10.16mm_Horizontal -> 9.09k 1% 1/4W
- RV1: value RV_Disc_D21mm_W5.5mm_P10.0mm -> S20K275 / V275LA20A
- RV2, RV3: value Potentiometer_Bourns_3296W_Vertical -> 3296W-1-102
- TP1, TP2, TP3, TP4, TP5, TP6, TP7, TP8: value TestPoint_THTPad_D2.0mm_Drill1.0mm -> Punto de prueba
- U1: value TO-220-5_Vertical -> LM2941CT/NOPB
- U2: value TO-220-5_Vertical -> LM2991T/NOPB
- U3: value TO-220-3_Vertical -> LM7805
- U4, U5: value DFN-10-1EP_3x3mm_P0.5mm_EP1.65x2.38mm -> LT3045EDD#TRPBF
- U6, U7: value DFN-12-1EP_3x3mm_P0.45mm_EP1.65x2.38mm -> LT3094EDD#PBF
Other:
- board text added: "+"
- board text added: "+12V"
- board text added: "+13V1"
- board text added: "+5V"
- board text added: "-12V"
- board text added: "-12V9"
- board text added: "GND"
- board text added: "SAM17 PSU v2"
- board text added: "U2 TAB = VRAW- ¡MICA!"
- board text added: "VRAW+"
- board text added: "VRAW-"
- board text added: "rev A - 2026-08-16"
