File: hardware/03-vco/kicad/sam17-vco.kicad_sch (KiCad schematic)
At the start: 136 parts, among them J1 PSU +12/G/G/-12, J2 Mazo digital IDC 2x6, U1 SSI2130, U10 74HC14, U11 L78L05, U12 LD1117S33TR, U13 TMP1075DGK, U14 24AA02E48, U2 SSI2130, U3 SSI2130, U4 SSI2130, U5 AD5686RBRUZ, U6 AD5686RBRUZ, U7 AD5686RBRUZ, U8 ADR4525BRZ, U9 TL074H

Commit message: Modulo 3: dos piezas por voz para que la salida deje de oscilar con un cable
Las que salieron del barrido de simulations/vco/iv_stage.py. Ocho componentes,
ningun cambio de topologia.

C_IV1-4, 33p C0G, en paralelo con R_IV: sin el, la capacidad del nodo MIXO_n con
los 10k forma un cero en la ganancia de ruido y el margen de fase se hunde. Es
el fallo clasico del amplificador de transimpedancia. Con 33p el polo del I/V
queda en 482 kHz, veinticuatro veces por encima del techo de audio: no cuesta
nada musicalmente. C0G obligatorio porque esta DENTRO del lazo.

R_OUT1-4, 220R, entre la salida del operacional y el jack: el TL074H esta
caracterizado con CL = 20 pF y un cable de instrumento son ~100 pF por metro;
con la Zo de 125 ohm eso es un polo dentro del lazo. Sin esta resistencia, 15 de
las 20 combinaciones del barrido oscilan en cuanto enchufas un cable. Va FUERA
del lazo -- la realimentacion se toma en IVO_n, antes -- asi que el cable no
entra en el lazo y no hay error de carga en continua, porque la entrada del
modulo 5 no consume. 220R contra sus ~100k es un divisor del 0.2 por mil.

La salida del opamp pasa a llamarse IVO_n y VOICE_OUT_n queda del lado del jack.
Esa es la frontera del lazo: lo que hay despues (jack, cable, modulo 5) queda
fuera y no puede desestabilizarlo.

Puertas: ERC 0 sobre la hoja regenerada desde cero. 144 componentes (eran 136,
+8 exactos) y 156 redes (eran 152, +4: IVO_1 a IVO_4). check_netlist.py verde
con todos sus invariantes. check_bom.py cruza 144 contra 144 fila por fila. El
diff del golden muestra exactamente los tres cambios buscados y ni una red mas.

Falta la placa. build_pcb.py necesita el jar de Freerouting y no esta en esta
maquina; el script no lo descarga a proposito. netdiff lo dice en rojo -- cuatro
redes y ocho huellas que estan en el esquematico y no en el cobre -- y ahi se
queda hasta que se rerutee. Sin cerrar y dicho, que es el Principio V.

Co-Authored-By: Claude Opus 5 (1M context) <noreply@anthropic.com>
Claude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
Parts:
- added C_IV1, C_IV2, C_IV3, C_IV4: 33p C0G, Capacitor_SMD:C_0805_2012Metric, symbol Device:C
- added R_OUT1, R_OUT2, R_OUT3, R_OUT4: 220R, Resistor_SMD:R_0805_2012Metric, symbol Device:R
Connections:
- net MIXO_1: now also C_IV1.1
- net MIXO_2: now also C_IV2.1
- net MIXO_3: now also C_IV3.1
- net MIXO_4: now also C_IV4.1
- net VOICE_OUT_1: now also R_OUT1.2; no longer R_IV1.2, U9.1
- net VOICE_OUT_2: now also R_OUT2.2; no longer R_IV2.2, U9.7
- net VOICE_OUT_3: now also R_OUT3.2; no longer R_IV3.2, U9.8
- net VOICE_OUT_4: now also R_OUT4.2; no longer R_IV4.2, U9.14
- new net IVO_1: C_IV1.2, R_IV1.2, R_OUT1.1, U9.1
- new net IVO_2: C_IV2.2, R_IV2.2, R_OUT2.1, U9.7
- new net IVO_3: C_IV3.2, R_IV3.2, R_OUT3.1, U9.8
- new net IVO_4: C_IV4.2, R_IV4.2, R_OUT4.1, U9.14
